Commit message: add VLP32 & VLP16 to gazebo

File: catkin_ws/src/gazebo/robot/bot/urdf/bot.xacro (robot description, xacro)
@@ -73,5 +73,5 @@
     </plugin>
   </gazebo>
-  <gazebo reference="camera">
+  <!--gazebo reference="camera">
     <material>Gazebo/Blue</material>
     <sensor name="camera_1" type="camera">
@@ -99,5 +99,5 @@
       </plugin>
     </sensor>
-  </gazebo>
+  </gazebo-->
   <link
     name="base_link">
@@ -352,5 +352,5 @@
       xyz="0 -1 0" />
   </joint>
-  <link name="camera">
+  <!--link name="camera">
     <collision>
       <origin rpy="0 0.1 0" xyz="0 0 0"/>
@@ -377,30 +377,47 @@
     <parent link="base_link"/>
     <child link="camera"/>
-  </joint>
-  <!--xacro:include filename="$(find velodyne_description)/urdf/VLP-16.urdf.xacro"/-->
-  <!--VLP-16 parent="base_link" name="velodyne" topic="/velodyne_points" hz="10" samples="440">
-    <origin xyz="0 0 0.05" rpy="0 0 0" />
-  </VLP-16-->
-  <xacro:include filename="$(find robot_sensors)/urdf/lidar_plugin.xacro" />
+  </joint-->
+  <!-- The VLP LIDAR xacro & dae source cloned from velodyne_simulator -->
+  <!-- https://bitbucket.org/DataspeedInc/velodyne_simulator/overview -->
   <xacro:if value="true">
-    <xacro:HDL32E_lidar parent="base_link"
-                        name="velodyne"
-                        topic="/velodyne_points"
-                        hz="8"
-                        samples="1800"
-                        min_range="0"
-                        max_range="100.0"
-                        min_angle="-3.14"
-                        max_angle="3.14"
-                        noise="0.01"
-                        gpu="true">
-      <origin xyz="0.3 0 0.3" rpy="0 0 -1.57" />
-    </xacro:HDL32E_lidar>
+    <xacro:include filename="$(find robot_sensors)/urdf/VLP-16.urdf.xacro"/>
+    <xacro:VLP-16   parent="base_link"
+                    name="velodyne_16"
+                    topic="/velodyne_points_16"
+                    hz="10"
+                    samples="1875"
+                    min_range="0"
+                    max_range="100.0"
+                    noise="0.01"
+                    gpu="true">
+      <origin xyz="0.3 0 0.5" rpy="0 0 0" />
+    </xacro:VLP-16>
   </xacro:if>
+  <xacro:if value="true">
+    <xacro:include filename="$(find robot_sensors)/urdf/HDL-32E.urdf.xacro" />
+    <xacro:HDL-32E  parent="base_link"
+                    name="velodyne_32"
+                    topic="/velodyne_points_32"
+                    hz="10"
+                    samples="2187"
+                    min_range="0"
+                    max_range="100.0"
+                    noise="0.01"
+                    gpu="true">
+        <origin xyz="0.3 0 0.35" rpy="0 0 -1.57" />
+    </xacro:HDL-32E>
+  </xacro:if>
+  <xacro:if value="true">
   <xacro:include filename="$(find robot_sensors)/urdf/rgbd_camera.xacro"/>
-  <xacro:if value="true">
-    <xacro:rgbd_camera name="rgbd" width="640" height="480" update_rate="20" pointCloudCutoffMax="6"/>
+    <xacro:rgbd_camera  name="rgbd"
+                        width="640"
+                        height="480"
+                        update_rate="20"
+                        min_distance="0.05"
+                        max_distance="100.0"
+                        pointCloudCutoff="0.6"
+                        pointCloudCutoffMax="100"/>
     <joint name="rgbd_camera_mount_joint" type="fixed">
-      <origin xyz="0.1 0 0.15" rpy="0 0.2618 0"/>
+      <origin xyz="0.3 0 0.62" rpy="0 0.0 0"/>
       <parent link="base_link"/>
       <child link="rgbd_link"/>

File: catkin_ws/src/gazebo/robot_sensors/urdf/HDL-32E.urdf.xacro (robot description, xacro)
@@ -1,6 +1,6 @@
 <?xml version="1.0"?>
-<robot xmlns:xacro="http://www.ros.org/wiki/xacro" name="HDL32E_lidar">
+<robot xmlns:xacro="http://www.ros.org/wiki/xacro" name="HDL-32E">
   <xacro:property name="M_PI" value="3.1415926535897931" />
-  <xacro:macro name="HDL32E_lidar" params="*origin parent:=base_link name:=velodyne topic:=/velodyne_points hz:=8 lasers:=32 samples:=2187 collision_range:=0.3 min_range:=0.9 max_range:=130.0 noise:=0.008 min_angle:=-${M_PI} max_angle:=${M_PI} gpu:=true">
+  <xacro:macro name="HDL-32E" params="*origin parent:=base_link name:=velodyne topic:=/velodyne_points hz:=10 lasers:=32 samples:=2187 collision_range:=0.3 min_range:=0.9 max_range:=130.0 noise:=0.008 min_angle:=-${M_PI} max_angle:=${M_PI} gpu:=true">
     <joint name="${name}_base_mount_joint" type="fixed">
       <xacro:insert_block name="origin" />
@@ -18,5 +18,5 @@
       <visual>
         <geometry>
-          <mesh filename="model://HDL32E/HDL32E_base.dae" />
+          <mesh filename="model://lidar/HDL32E_base.dae" />
         </geometry>
       </visual>
@@ -42,5 +42,5 @@
         <origin xyz="0 0 -0.09081" rpy="0 0 0" />
         <geometry>
-          <mesh filename="model://HDL32E/HDL32E_scan.dae" />
+          <mesh filename="model://lidar/HDL32E_scan.dae" />
         </geometry>
       </visual>
@@ -49,5 +49,5 @@
     <gazebo reference="${name}">
       <xacro:if value="${gpu}">
-        <sensor type="gpu_ray" name="${name}_HDL32E">
+        <sensor type="gpu_ray" name="${name}-HDL32E">
           <pose>0 0 0 0 0 0</pose>
           <visualize>false</visualize>
@@ -89,5 +89,5 @@
       </xacro:if>
       <xacro:unless value="${gpu}">
-        <sensor type="ray" name="${name}_HDL32E">
+        <sensor type="ray" name="${name}-HDL32E">
           <pose>0 0 0 0 0 0</pose>
           <visualize>false</visualize>

File: catkin_ws/src/gazebo/robot_sensors/urdf/rgbd_camera.xacro (robot description, xacro)
@@ -28,6 +28,6 @@
                params="name:=camera
                        robot_namespace:=/
-                       width:=320
-                       height:=240
+                       width:=640
+                       height:=480
                        update_rate:=30.0
                        min_distance:=0.05

Commit message: add world to empty world

File: catkin_ws/src/gazebo/robot/bot/urdf/bot.xacro (robot description, xacro)
@@ -391,5 +391,5 @@
                     noise="0.01"
                     gpu="true">
-      <origin xyz="0.3 0 0.5" rpy="0 0 0" />
+      <origin xyz="0.1 0 0.3" rpy="0 0 0" />
     </xacro:VLP-16>
   </xacro:if>
@@ -405,5 +405,5 @@
                     noise="0.01"
                     gpu="true">
-        <origin xyz="0.3 0 0.35" rpy="0 0 -1.57" />
+        <origin xyz="0.1 0 0.15" rpy="0 0 -1.57" />
     </xacro:HDL-32E>
   </xacro:if>
@@ -419,5 +419,5 @@
                         pointCloudCutoffMax="100.0"/>
     <joint name="rgbd_camera_mount_joint" type="fixed">
-      <origin xyz="0.3 0 0.62" rpy="0 0.0 0"/>
+      <origin xyz="0.1 0 0.42" rpy="0 0.0 0"/>
       <parent link="base_link"/>
       <child link="rgbd_link"/>
